File: UsbSound.kicad_pcb (KiCad board)
At the start: 0 parts

Commit message: First rev of board is done
If at first you don't succeed... try...try...try...try...try...try...try...try...
Parts:
- added C1: 10u, Capacitor_SMD:C_1206_3216Metric, F.Cu at (106.5, 73.7)
- added C10: 100n, Capacitor_SMD:C_1206_3216Metric, F.Cu at (129.5, 89.7)
- added C11: 100n, Capacitor_SMD:C_1206_3216Metric, F.Cu at (114.9, 96.1)
- added C12: 100n, Capacitor_SMD:C_1206_3216Metric, F.Cu at (117.7, 105.6)
- added C13: 100n, Capacitor_SMD:C_1206_3216Metric, F.Cu at (132.4, 104.4)
- added C14: 1u, Capacitor_SMD:C_1206_3216Metric, F.Cu at (148.5, 95.0)
- added C15: 10n, Capacitor_SMD:C_1206_3216Metric, F.Cu at (148.5, 100.2)
- added C16: 47u, Capacitor_SMD:C_1206_3216Metric, F.Cu at (159.3, 86.7)
- added C17: 22pF, Capacitor_SMD:C_1206_3216Metric, F.Cu at (146.4, 83.1)
- added C18: 0u1, Capacitor_SMD:C_1206_3216Metric, F.Cu at (142.3, 81.0)
- added C19: 2u2, Capacitor_SMD:C_1206_3216Metric, F.Cu at (114.8, 102.0)
- added C2: 10u, Capacitor_SMD:C_1206_3216Metric, F.Cu at (111.6, 63.1)
- added C20: 2u2, Capacitor_SMD:C_1206_3216Metric, F.Cu at (130.1, 106.9)
- added C21: 2700pF, Capacitor_SMD:C_1206_3216Metric, F.Cu at (136.5, 77.4)
- added C22: 0u1, Capacitor_SMD:C_1206_3216Metric, F.Cu at (133.6, 82.1)
- added C23: 12p, Capacitor_SMD:C_1206_3216Metric, F.Cu at (121.0, 85.3)
- added C24: 12p, Capacitor_SMD:C_1206_3216Metric, F.Cu at (110.7, 85.3)
- added C25: 22pF, Capacitor_SMD:C_1206_3216Metric, F.Cu at (125.3, 75.8)
- added C26: 12p, Capacitor_SMD:C_1206_3216Metric, F.Cu at (175.6, 114.3)
- added C27: 12p, Capacitor_SMD:C_1206_3216Metric, F.Cu at (166.7, 114.0)
- added C28: 0u1, Capacitor_SMD:C_1206_3216Metric, F.Cu at (127.4, 71.9)
- added C29: 0.1u, Capacitor_SMD:C_1206_3216Metric, F.Cu at (162.8, 100.8)
- added C3: 10u, Capacitor_SMD:C_1206_3216Metric, F.Cu at (98.1, 77.3)
- added C30: 10u, Capacitor_SMD:C_1206_3216Metric, F.Cu at (162.8, 104.8)
- added C31: 2700pF, Capacitor_SMD:C_1206_3216Metric, F.Cu at (188.4, 72.3)
- added C32: 10u, Capacitor_SMD:C_1206_3216Metric, F.Cu at (159.3, 84.3)
- added C33: 0.1u, Capacitor_SMD:C_1206_3216Metric, F.Cu at (166.8, 87.9)
- added C34: 10u, Capacitor_SMD:C_1206_3216Metric, F.Cu at (172.4, 87.9)
- added C35: 0.1u, Capacitor_SMD:C_1206_3216Metric, F.Cu at (153.1, 87.9)
- added C36: 10u, Capacitor_SMD:C_1206_3216Metric, F.Cu at (150.6, 87.9)
- added C37: 0u1, Capacitor_SMD:C_1206_3216Metric, F.Cu at (193.5, 74.9)
- added C38: 22pF, Capacitor_SMD:C_1206_3216Metric, F.Cu at (186.5, 83.6)
- added C39: 0u1, Capacitor_SMD:C_1206_3216Metric, F.Cu at (182.6, 81.2)
- added C4: 10u, Capacitor_SMD:C_1206_3216Metric, F.Cu at (106.2, 78.7)
- added C40: 2700pF, Capacitor_SMD:C_1206_3216Metric, F.Cu at (175.7, 77.9)
- added C41: 0u1, Capacitor_SMD:C_1206_3216Metric, F.Cu at (173.2, 82.3)
- added C42: 22pF, Capacitor_SMD:C_1206_3216Metric, F.Cu at (164.7, 75.9)
- added C43: 0u1, Capacitor_SMD:C_1206_3216Metric, F.Cu at (166.9, 71.9)
- added C5: 2700pF, Capacitor_SMD:C_1206_3216Metric, F.Cu at (147.9, 71.9)
- added C6: 1u, Capacitor_SMD:C_1206_3216Metric, F.Cu at (113.9, 90.3)
- added C7: 10n, Capacitor_SMD:C_1206_3216Metric, F.Cu at (118.0, 90.3)
- added C8: 0u1, Capacitor_SMD:C_1206_3216Metric, F.Cu at (153.9, 75.3)
- added C9: 4u7, Capacitor_SMD:C_1206_3216Metric, F.Cu at (129.5, 87.2)
- added D1: B5819W, Diode_SMD:D_SOD-123, F.Cu at (101.6, 68.9)
- added D2: B5819W, Diode_SMD:D_SOD-123, F.Cu at (108.1, 68.4)
- added D3: Red, LED_SMD:LED_1206_3216Metric, F.Cu at (111.1, 118.1)
- added F1: 250mA, Fuse:Fuse_1206_3216Metric, F.Cu at (103.2, 63.2)
- added FB1: 600 @ 600MHz, Inductor_SMD:L_0805_2012Metric, F.Cu at (108.0, 63.0)
- added J1: SWD, Connector_PinHeader_1.27mm:PinHeader_2x05_P1.27mm_Vertical_SMD, F.Cu at (90.6, 96.7)
- added J2: USB_B, Connector_USB:USB_A_Molex_67643_Horizontal, F.Cu at (96.5, 53.6)
- added J3: XLR_L, Connector_Audio:Jack_XLR_Neutrik_NC3MAH_Horizontal, F.Cu at (143.2, 62.6)
- added J4: XLR_R, Connector_Audio:Jack_XLR_Neutrik_NC3MAH_Horizontal, F.Cu at (182.4, 62.6)
- added L1: 10u, Inductor_SMD:L_1206_3216Metric, F.Cu at (101.4, 73.8)
- added L2: 39n, Inductor_SMD:L_0402_1005Metric, F.Cu at (110.4, 91.8)
- added L3: 39n, Inductor_SMD:L_1206_3216Metric, F.Cu at (143.2, 96.6)
- added R1: 47k, Resistor_SMD:R_1206_3216Metric, F.Cu at (116.6, 75.5)
- added R10: 27, Resistor_SMD:R_1206_3216Metric, F.Cu at (157.8, 109.7)
- added R11: 27, Resistor_SMD:R_1206_3216Metric, F.Cu at (154.0, 109.7)
- added R12: 10k, Resistor_SMD:R_1206_3216Metric, F.Cu at (167.6, 94.5)
- added R13: 820, Resistor_SMD:R_1206_3216Metric, F.Cu at (136.5, 73.8)
- added R14: 0, Resistor_SMD:R_1206_3216Metric, F.Cu at (123.5, 89.3)
- added R15: 0, Resistor_SMD:R_1206_3216Metric, F.Cu at (165.5, 110.5)
- added R16: 820, Resistor_SMD:R_1206_3216Metric, F.Cu at (184.5, 72.3)
- added R17: 4k7, Resistor_SMD:R_1206_3216Metric, F.Cu at (137.2, 93.4)
- added R18: 4k7, Resistor_SMD:R_1206_3216Metric, F.Cu at (133.4, 93.4)
- added R19: 820, Resistor_SMD:R_1206_3216Metric, F.Cu at (175.7, 73.9)
- added R2: 15k, Resistor_SMD:R_1206_3216Metric, F.Cu at (116.5, 79.7)
- added R3: 270, Resistor_SMD:R_1206_3216Metric, F.Cu at (111.3, 79.7)
- added R4: 100k, Resistor_SMD:R_1206_3216Metric, F.Cu at (113.9, 69.6)
- added R5: 68k, Resistor_SMD:R_1206_3216Metric, F.Cu at (118.8, 70.8)
- added R6: 820, Resistor_SMD:R_1206_3216Metric, F.Cu at (144.4, 71.9)
- added R7: 2k2, Resistor_SMD:R_1206_3216Metric, F.Cu at (105.4, 118.1)
- added R8: 10k, Resistor_SMD:R_1206_3216Metric, F.Cu at (85.4, 76.9)
- added R9: 27, Resistor_SMD:R_1206_3216Metric, F.Cu at (161.6, 109.7)
- added SW1: BOOT_SELECT, Button_Switch_SMD:SW_SPDT_PCM12, F.Cu at (78.2, 76.2)
- added U1: MP2359-LF-Z, Package_TO_SOT_SMD:SOT-23-6, F.Cu at (112.4, 73.7)
- added U2: USBLC6-2SC6, Package_TO_SOT_SMD:SOT-23-6, F.Cu at (93.0, 67.6)
- added U3: NE5534, Package_SO:SOIC-8-1EP_3.9x4.9mm_P1.27mm_EP2.29x3mm, F.Cu at (147.2, 78.8)
- added U4: PCM1795DB, symbols:SOP65P780X200-28N, F.Cu at (159.7, 93.1)
- added U5: STM32F405RGT6, Package_QFP:LQFP-64_10x10mm_P0.5mm, F.Cu at (124.3, 98.9)
- added U6: NE5534, Package_SO:SOIC-8-1EP_3.9x4.9mm_P1.27mm_EP2.29x3mm, F.Cu at (129.6, 76.8)
- added U7: NE5534, Package_SO:SOIC-8-1EP_3.9x4.9mm_P1.27mm_EP2.29x3mm, F.Cu at (187.5, 79.1)
- added U8: NE5534, Package_SO:SOIC-8-1EP_3.9x4.9mm_P1.27mm_EP2.29x3mm, F.Cu at (169.1, 76.8)
- added Y1: 16MHz, Crystal:Crystal_SMD_3225-4Pin_3.2x2.5mm, F.Cu at (115.9, 85.5)
- added Y2: 36.864MHz, Crystal:Crystal_SMD_3225-4Pin_3.2x2.5mm, F.Cu at (171.3, 111.6)
Routing:
- net +3V3: track 0.00 -> 252.3 mm, vias 0 -> 17
- net +5VA: track 0.00 -> 153.7 mm, vias 0 -> 8
- net -5VA: track 0.00 -> 97.9 mm, vias 0 -> 4
- net +5V: track 0.00 -> 88.0 mm, vias 0 -> 2
- net SWO: track 0.00 -> 80.8 mm, vias 0 -> 2
- net SWCLK: track 0.00 -> 72.7 mm
- net USB_D+: track 0.00 -> 70.2 mm
- net USB_D-: track 0.00 -> 68.1 mm
- net BOOT0: track 0.00 -> 66.8 mm, vias 0 -> 2
- net POUTR-: track 0.00 -> 65.5 mm
- net POUTR+: track 0.00 -> 60.3 mm
- net SWDIO: track 0.00 -> 55.3 mm
- net GND: track 0.00 -> 54.9 mm, vias 0 -> 157
- net POUTL-: track 0.00 -> 54.8 mm
- net I2C1_SCL: track 0.00 -> 52.2 mm, vias 0 -> 2
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- added copper zone on F.Cu, net GND
- added copper zone on In1.Cu, net GND
Other:
- board outline added: 121.6 x 79.8 mm
- copper layers 0 -> 4
- board text added: "BOOT"
- board text added: "JLCJLCJLCJLC"
- board text added: "Left"
- board text added: "Left+"
- board text added: "Left-"
- board text added: "Low Expectations External Sound Card (C) Steve Syfuhs 2021 Rev 0.1 - If at first you don't succeed."
- board text added: "RUN"
- board text added: "Right"
- board text added: "Right+"
- board text added: "Right-"
