File: UsbSound.kicad_sch (KiCad schematic)
At the start: 82 parts

Commit message: fixup electrical rules and stupid grids
Added crystal for PCM clock.
Added footprints for most components.
Parts:
- removed R?: 27, symbol Device:R_Small
- added C13, C17: 12p, Capacitor_SMD:C_1206_3216Metric, symbol Device:C_Small
- added R11: 0, symbol Device:R_Small
- added Y2: 36.864MHz, symbol Device:Crystal_GND24_Small
- C1, C10, C12, C14, C16, C18, C19, C2, C20, C21, C22, C23, C24, C25, C26, C27, C28, C29, C3, C30, C31, C32, C33, C34, C35, C36, C37, C38, C39, C4, C40, C41, C42, C43, C5, C6, C7, C8: renamed from C?; footprint (none) -> Capacitor_SMD:C_1206_3216Metric
- C9: renamed from C?; footprint Capacitor_SMD:C_0402_1005Metric -> Capacitor_SMD:C_1206_3216Metric
- D3: renamed from D?; footprint (none) -> Diode_SMD:D_SOD-123
- gave numbers to parts that had none: 41
Connections:
- net +3V3: now also C13.1, Y2.1
- net GND: now also C13.2, C17.2, Y2.2, Y2.4
- net at R13.2: now also R14.1
- net PCMSCK: now reaches U4.7 (SCL)
- net PCMSCK: now also R11.1
- net I2S3_MCK: no longer names the net of U2.38 (PC7)
- net I2S3_WS: no longer names the net of U2.20 (PA4)
- new net: C17.1, R11.2, Y2.3
- no-connect marks 40 -> 47
Other:
- moved on the sheet: C12, C14, C18, C20, C21, C22, C24

Commit message: First rev of board is done
If at first you don't succeed... try...try...try...try...try...try...try...try...
Parts:
- removed J1: USB_B_Micro, SchmillipKiCADLibrary:USB_MICRO_B_101181930001LF, symbol STM32F4_REV2-rescue:USB_B_Micro-Connector
- added J2: USB_B, Connector_USB:USB_A_Molex_67643_Horizontal, symbol Connector:USB_B
- C7: renamed from C11; footprint Capacitor_SMD:C_0402_1005Metric -> Capacitor_SMD:C_1206_3216Metric
- D3: renamed from D1; footprint (none) -> LED_SMD:LED_1206_3216Metric
- J3, J4: footprint (none) -> Connector_Audio:Jack_XLR_Neutrik_NC3MAH_Horizontal
- L1: renamed from L3; footprint (none) -> Inductor_SMD:L_1206_3216Metric
- L3: renamed from L2; footprint (none) -> Inductor_SMD:L_1206_3216Metric
- R1: renamed from R12; footprint (none) -> Resistor_SMD:R_1206_3216Metric
- R10: renamed from R9; footprint (none) -> Resistor_SMD:R_1206_3216Metric
- R11: renamed from R10; footprint (none) -> Resistor_SMD:R_1206_3216Metric
- R12: renamed from R15; footprint (none) -> Resistor_SMD:R_1206_3216Metric
- R13: renamed from R18; footprint (none) -> Resistor_SMD:R_1206_3216Metric
- R14: renamed from R1; footprint (none) -> Resistor_SMD:R_1206_3216Metric
- R15: renamed from R11; footprint (none) -> Resistor_SMD:R_1206_3216Metric
- R16: renamed from R17; footprint (none) -> Resistor_SMD:R_1206_3216Metric
- R17: renamed from R4; footprint (none) -> Resistor_SMD:R_1206_3216Metric
- R18: renamed from R5; footprint (none) -> Resistor_SMD:R_1206_3216Metric
- R19: renamed from R16; footprint (none) -> Resistor_SMD:R_1206_3216Metric
- R2: renamed from R13; footprint (none) -> Resistor_SMD:R_1206_3216Metric
- R3: renamed from R14; footprint (none) -> Resistor_SMD:R_1206_3216Metric
- R4: renamed from R6; footprint (none) -> Resistor_SMD:R_1206_3216Metric
- R5: renamed from R7; footprint (none) -> Resistor_SMD:R_1206_3216Metric
- R6: renamed from R19; footprint (none) -> Resistor_SMD:R_1206_3216Metric
- R7: renamed from R2; footprint (none) -> Resistor_SMD:R_1206_3216Metric
- R8: renamed from R3; footprint (none) -> Resistor_SMD:R_1206_3216Metric
- R9: renamed from R8; footprint (none) -> Resistor_SMD:R_1206_3216Metric
- SW1: footprint (none) -> Button_Switch_SMD:SW_SPDT_PCM12
- U1: renamed from U3; footprint (none) -> Package_TO_SOT_SMD:SOT-23-6
- U3: renamed from U8; footprint (none) -> Package_SO:SOIC-8-1EP_3.9x4.9mm_P1.27mm_EP2.29x3mm
- U4: footprint SOP65P780X200-28N -> symbols:SOP65P780X200-28N
- U6: renamed from U7; footprint (none) -> Package_SO:SOIC-8-1EP_3.9x4.9mm_P1.27mm_EP2.29x3mm
- U7: renamed from U6; footprint (none) -> Package_SO:SOIC-8-1EP_3.9x4.9mm_P1.27mm_EP2.29x3mm
- U8: renamed from U5; footprint (none) -> Package_SO:SOIC-8-1EP_3.9x4.9mm_P1.27mm_EP2.29x3mm
- Y1, Y2: footprint (none) -> Crystal:Crystal_SMD_3225-4Pin_3.2x2.5mm
- renumbered C27 to C1, C3 to C10, C4 to C11, C6 to C12, C7 to C13, C16 to C14, C19 to C15, C23 to C16, C43 to C17, C35 to C18, C8 to C19, C15 to C2, C10 to C20, C38 to C21, C30 to C22, C2 to C23, C5 to C24, C42 to C25, C13 to C26, C17 to C27, C34 to C28, C22 to C29, C25 to C3, C24 to C30, C37 to C31, C12 to C32, C14 to C33, C18 to C34, C20 to C35, C21 to C36, C29 to C37, C41 to C38, C33 to C39, C26 to C4, C36 to C40, C28 to C41, C40 to C42, C32 to C43, C39 to C5, C9 to C6, C31 to C8, C1 to C9, D2 to D1, D3 to D2, J2 to J1, L1 to L2, U1 to U2, U2 to U5
Connections:
- net +5V: now also J2.1 (VBUS)
- net +5VA: now also U4.23 (VCOMR); no longer U4.21 (VCC1)
- net GND: now also J2.5 (Shield)
- net USB_CONN_D+: now also J2.3 (D+)
- net USB_CONN_D-: now also J2.2 (D-)
- net ZEROL: now also U5.57 (PB5); no longer U5.29 (PB10)
- net ZEROR: now also U5.56 (PB4); no longer U5.30 (PB11)
- net at C16.2, U4.22 (VCOML): now also U4.21 (VCC1); no longer U4.23 (VCOMR)
- no-connect marks 47 -> 46
Other:
- moved on the sheet: C16

Commit message: Added -5v rail because I'm an idiot and forgot it
Parts:
- added C2, C4: 10u, Capacitor_SMD:C_1206_3216Metric, symbol Device:C_Small
- added U2: ICL7660, Package_SO:SOIC-8-1EP_3.9x4.9mm_P1.27mm_EP2.29x3mm, symbol Regulator_SwitchedCapacitor:ICL7660
- J2: footprint Connector_USB:USB_A_Molex_67643_Horizontal -> Connector_USB:USB_B_Lumberg_2411_02_Horizontal
- renumbered C8 to C10, C9 to C11, C10 to C12, C11 to C13, C12 to C14, C13 to C15, C14 to C16, C15 to C17, C16 to C18, C17 to C19, C18 to C20, C19 to C21, C20 to C22, C21 to C23, C22 to C24, C23 to C25, C24 to C26, C25 to C27, C26 to C28, C27 to C29, C2 to C3, C28 to C30, C29 to C31, C30 to C32, C31 to C33, C32 to C34, C33 to C35, C34 to C36, C35 to C37, C36 to C38, C37 to C39, C38 to C40, C39 to C41, C40 to C42, C41 to C43, C42 to C44, C43 to C45, C3 to C5, C4 to C6, C5 to C7, C6 to C8, C7 to C9, U2 to U3, U3 to U4, U4 to U5, U5 to U6, U6 to U7, U7 to U8, U8 to U9
Connections:
- net +5V: now also U2.8 (V+)
- net -5VA: now also C2.1, U2.5 (VOUT)
- net GND: now also C2.2, U2.3 (GND)
- new net: C4.2, U2.2 (CAP+)
- new net: C4.1, U2.4 (CAP-)
- no-connect marks 46 -> 48

Commit message: Fixing models
Parts:
- removed U1: MP2359-LF-Z, Package_TO_SOT_SMD:SOT-23-6, symbol Custom:MP2359-LF-Z
- added U1: XRP7659, Package_SO:TSOP-6_1.65x3.05mm_P0.95mm, symbol Custom:XRP7659
Connections:
- net BUCK_BST: now also U1.1 (BS)
- net BUCK_EN: now also U1.4 (EN)
- net BUCK_FB: now also U1.3 (FB)
- net BUCK_IN: now also U1.5 (VIN)
- net BUCK_SW: now also U1.6 (SW)
- net GND: now also U1.2 (GND)
Changed lines of the file:
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@@
   (junction (at 47.625 78.105) (diameter 1.016) (color 0 0 0 0))
   (junction (at 47.625 85.725) (diameter 1.016) (color 0 0 0 0))
-  (junction (at 63.5 108.331) (diameter 0.9144) (color 0 0 0 0))
   (junction (at 67.945 69.85) (diameter 1.016) (color 0 0 0 0))
   (junction (at 67.945 76.2) (diameter 1.016) (color 0 0 0 0))
-  (junction (at 72.39 118.618) (diameter 0.9144) (color 0 0 0 0))
   (junction (at 74.93 26.67) (diameter 1.016) (color 0 0 0 0))
   (junction (at 74.93 31.75) (diameter 1.016) (color 0 0 0 0))
@@
   (junction (at 209.55 88.138) (diameter 0.9144) (color 0 0 0 0))
   (junction (at 215.265 47.625) (diameter 0.9144) (color 0 0 0 0))
-  (junction (at 219.456 88.138) (diameter 0.9144) (color 0 0 0 0))
   (junction (at 223.52 47.625) (diameter 0.9144) (color 0 0 0 0))
   (junction (at 241.3 227.838) (diameter 0.9144) (color 0 0 0 0))
@@
     (stroke (width 0) (type solid) (color 0 0 0 0))
   )
-  (wire (pts (xy 59.309 108.331) (xy 63.5 108.331))
-    (stroke (width 0) (type solid) (color 0 0 0 0))
-  )
   (wire (pts (xy 63.5 108.331) (xy 78.74 108.331))
     (stroke (width 0) (type solid) (color 0 0 0 0))
@@
     (stroke (width 0) (type solid) (color 0 0 0 0))
   )
-  (wire (pts (xy 72.39 118.491) (xy 72.39 118.618))
-    (stroke (width 0) (type solid) (color 0 0 0 0))
-  )
-  (wire (pts (xy 72.39 118.618) (xy 72.39 119.761))
+  (wire (pts (xy 72.39 118.618) (xy 72.39 120.142))
     (stroke (width 0) (type solid) (color 0 0 0 0))
   )
@@
     (stroke (width 0) (type solid) (color 0 0 0 0))
   )
-  (wire (pts (xy 209.55 88.138) (xy 219.456 88.138))
+  (wire (pts (xy 209.55 88.138) (xy 214.122 88.138))
     (stroke (width 0) (type solid) (color 0 0 0 0))
   )
@@
     (stroke (width 0) (type solid) (color 0 0 0 0))
   )
-  (wire (pts (xy 219.456 88.138) (xy 220.726 88.138))
-    (stroke (width 0) (type solid) (color 0 0 0 0))
-  )
-  (wire (pts (xy 220.726 88.138) (xy 220.726 87.63))
-    (stroke (width 0) (type solid) (color 0 0 0 0))
-  )
   (wire (pts (xy 223.52 42.545) (xy 223.52 47.625))
     (stroke (width 0) (type solid) (color 0 0 0 0))
@@
     )
   )
-  (global_label "BUCK_BST" (shape input) (at 184.15 36.83 0)
+  (global_label "BUCK_BST" (shape input) (at 185.166 36.83 0)
     (effects (font (size 1.27 1.27)) (justify left))
-    (property "Intersheet References" "${INTERSHEET_REFS}" (id 0) (at 196.1183 36.7506 0)
+    (property "Intersheet References" "${INTERSHEET_REFS}" (id 0) (at 197.1343 36.7506 0)
       (effects (font (size 1.27 1.27)) (justify left) hide)
     )
   )
-  (global_label "BUCK_SW" (shape input) (at 184.15 39.37 0)
+  (global_label "BUCK_SW" (shape input) (at 185.166 39.37 0)
     (effects (font (size 1.27 1.27)) (justify left))
-    (property "Intersheet References" "${INTERSHEET_REFS}" (id 0) (at 195.3321 39.2906 0)
+    (property "Intersheet References" "${INTERSHEET_REFS}" (id 0) (at 196.3481 39.2906 0)
       (effects (font (size 1.27 1.27)) (justify left) hide)
     )
   )
-  (global_label "BUCK_FB" (shape input) (at 184.15 41.91 0)
+  (global_label "BUCK_FB" (shape input) (at 185.166 41.91 0)
     (effects (font (size 1.27 1.27)) (justify left))
-    (property "Intersheet References" "${INTERSHEET_REFS}" (id 0) (at 195.0298 41.8306 0)
+    (property "Intersheet References" "${INTERSHEET_REFS}" (id 0) (at 196.0458 41.8306 0)
       (effects (font (size 1.27 1.27)) (justify left) hide)
     )
@@
     (pin "1")
   )
-  (symbol (lib_id "power:+5VA") (at 220.726 87.63 0) (unit 1)
+  (symbol (lib_id "power:+5VA") (at 214.122 88.138 0) (unit 1)
+    (in_bom yes) (on_board yes)
+    (property "Reference" "#PWR0102" (id 0) (at 214.122 91.948 0)
+      (effects (font (size 1.27 1.27)) hide)
+    )
+    (property "Value" "+5VA" (id 1) (at 214.4903 83.8136 0))
+    (property "Footprint" "" (id 2) (at 214.122 88.138 0)
+      (effects (font (size 1.27 1.27)) hide)
+    )
+    (property "Datasheet" "" (id 3) (at 214.122 88.138 0)
+      (effects (font (size 1.27 1.27)) hide)
+    )
+    (pin "1")
+  )
+  (symbol (lib_id "power:+5VA") (at 219.456 88.138 0) (unit 1)
     (in_bom yes) (on_board yes)
-    (property "Reference" "#PWR035" (id 0) (at 220.726 91.44 0)
+    (property "Reference" "#PWR035" (id 0) (at 219.456 91.948 0)
       (effects (font (size 1.27 1.27)) hide)
     )
-    (property "Value" "+5VA" (id 1) (at 221.0943 83.3056 0))
-    (property "Footprint" "" (id 2) (at 220.726 87.63 0)
+    (property "Value" "+5VA" (id 1) (at 219.8243 83.8136 0))
+    (property "Footprint" "" (id 2) (at 219.456 88.138 0)
       (effects (font (size 1.27 1.27)) hide)
     )
-    (property "Datasheet" "" (id 3) (at 220.726 87.63 0)
+    (property "Datasheet" "" (id 3) (at 219.456 88.138 0)
       (effects (font (size 1.27 1.27)) hide)
     )
@@
     (pin "1")
   )
-  (symbol (lib_id "power:GND") (at 72.39 119.761 0) (unit 1)
+  (symbol (lib_id "power:GND") (at 72.39 120.142 0) (unit 1)
     (in_bom yes) (on_board yes)
-    (property "Reference" "#PWR047" (id 0) (at 72.39 126.111 0)
+    (property "Reference" "#PWR047" (id 0) (at 72.39 126.492 0)
       (effects (font (size 1.27 1.27)) hide)
     )
-    (property "Value" "GND" (id 1) (at 72.517 124.1552 0))
-    (property "Footprint" "" (id 2) (at 72.39 119.761 0)
+    (property "Value" "GND" (id 1) (at 72.517 124.5362 0))
+    (property "Footprint" "" (id 2) (at 72.39 120.142 0)
       (effects (font (size 1.27 1.27)) hide)
     )
-    (property "Datasheet" "" (id 3) (at 72.39 119.761 0)
+    (property "Datasheet" "" (id 3) (at 72.39 120.142 0)
       (effects (font (size 1.27 1.27)) hide)
     )
@@
     (pin "9")
   )
-  (symbol (lib_id "Custom:MP2359-LF-Z") (at 177.8 36.195 0) (unit 1)
+  (symbol (lib_id "Custom:XRP7659") (at 177.8 32.766 0) (unit 1)
     (in_bom yes) (on_board yes)
-    (property "Reference" "U1" (id 0) (at 177.8 31.2482 0))
-    (property "Value" "MP2359-LF-Z" (id 1) (at 177.8 33.5469 0))
-    (property "Footprint" "Package_TO_SOT_SMD:SOT-23-6" (id 2) (at 176.53 36.195 0)
+    (property "Reference" "U1" (id 0) (at 178.308 31.248 0))
+    (property "Value" "XRP7659" (id 1) (at 178.308 33.5469 0))
+    (property "Footprint" "Package_SO:TSOP-6_1.65x3.05mm_P0.95mm" (id 2) (at 177.8 32.766 0)
       (effects (font (size 1.27 1.27)) hide)
     )
-    (property "Datasheet" "" (id 3) (at 176.53 36.195 0)
+    (property "Datasheet" "" (id 3) (at 177.8 32.766 0)
       (effects (font (size 1.27 1.27)) hide)
     )
@@
       (reference "#PWR0101") (unit 1) (value "-5VA") (footprint "")
     )
+    (path "/7bb05d06-fb7f-4e3b-a205-3258461d7034"
+      (reference "#PWR0102") (unit 1) (value "+5VA") (footprint "")
+    )
     (path "/d2805692-0fa1-4892-92c5-4fa7c1a7131f"
       (reference "C1") (unit 1) (value "10u") (footprint "Capacitor_SMD:C_1206_3216Metric")
@@
       (reference "SW1") (unit 1) (value "BOOT_SELECT") (footprint "Button_Switch_SMD:SW_SPDT_PCM12")
     )
-    (path "/7f825545-ed6f-4739-a670-3634abee2a0a"
-      (reference "U1") (unit 1) (value "MP2359-LF-Z") (footprint "Package_TO_SOT_SMD:SOT-23-6")
+    (path "/af092c54-379a-4c02-8b14-602001985ad0"
+      (reference "U1") (unit 1) (value "XRP7659") (footprint "Package_SO:TSOP-6_1.65x3.05mm_P0.95mm")
     )
     (path "/a2a290cf-1f4c-4a10-bbcd-07ef7224b068"

Commit message: Maybe fixed clock path. Moved some power routes to avoid analog signal.
Added some additional silkscreen for useful text.
Connections:
- net I2S3_CK: no longer R11.1
- net I2S3_MCK: now reaches U6.38 (PC7)
- net I2S3_MCK: now also R11.1
- no-connect marks 48 -> 47
Changed lines of the file:
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@@
   (no_connect (at 78.74 154.051))
   (no_connect (at 78.74 156.591))
-  (no_connect (at 78.74 159.131))
   (no_connect (at 78.74 161.671))
   (no_connect (at 78.74 164.211))
@@
     )
   )
+  (global_label "I2S3_MCK" (shape input) (at 78.74 159.131 180)
+    (effects (font (size 1.27 1.27)) (justify right))
+    (property "Intersheet References" "${INTERSHEET_REFS}" (id 0) (at 67.1345 159.0516 0)
+      (effects (font (size 1.27 1.27)) (justify right) hide)
+    )
+  )
   (global_label "I2S3_CK" (shape input) (at 78.74 166.751 180)
     (effects (font (size 1.27 1.27)) (justify right))
@@
     )
   )
-  (global_label "I2S3_CK" (shape input) (at 150.114 108.458 180)
-    (effects (font (size 1.27 1.27)) (justify right))
-    (property "Intersheet References" "${INTERSHEET_REFS}" (id 0) (at 94.234 -52.832 0)
-      (effects (font (size 1.27 1.27)) hide)
-    )
-  )
+  (global_label "I2S3_MCK" (shape input) (at 150.114 108.458 180)
+    (effects (font (size 1.27 1.27)) (justify right))
+    (property "Intersheet References" "${INTERSHEET_REFS}" (id 0) (at 138.5085 108.3786 0)
+      (effects (font (size 1.27 1.27)) (justify right) hide)
+    )
+  )

Commit message: Added GPIO pin header for future testing
Parts:
- added D4: Red, LED_SMD:LED_1206_3216Metric, symbol Device:LED_Small
- added J5: SWD, Connector_PinHeader_1.27mm:PinHeader_2x05_P1.27mm_Vertical_SMD, symbol Connector_Generic:Conn_02x05_Odd_Even
- added R20: 2k2, Resistor_SMD:R_1206_3216Metric, symbol Device:R_Small
Connections:
- net GND: now also R20.2
- net RVA-: now reaches C40.2, U8.5 (COMP)
- net RVAC-: now reaches C40.1, U8.8 (C/B)
- net LED_STATUS1: now reaches U6.15 (PA1)
- net LED_STATUS1: now also D3.2 (A)
- net VCAP1: now reaches C21.1, U6.31 (VCAP_1)
- net GPIO_1: now reaches U6.33 (PB12)
- net GPIO_1: now also J5.1 (Pin_1)
- net GPIO_2: now reaches U6.34 (PB13)
- net GPIO_2: now also J5.2 (Pin_2)
- net GPIO_3: now reaches U6.35 (PB14)
- net GPIO_3: now also J5.3 (Pin_3)
- net GPIO_4: now reaches U6.36 (PB15)
- net GPIO_4: now also J5.4 (Pin_4)
- net GPIO_5: now reaches U6.37 (PC6)
- net GPIO_5: now also J5.5 (Pin_5)
- net GPIO_6: now reaches U6.39 (PC8)
- net GPIO_6: now also J5.6 (Pin_6)
- net GPIO_7: now reaches U6.40 (PC9)
- net GPIO_7: now also J5.7 (Pin_7)
- net GPIO_8: now reaches U6.41 (PA8)
- net GPIO_8: now also J5.8 (Pin_8)
- net GPIO_9: now reaches U6.42 (PA9)
- net GPIO_9: now also J5.9 (Pin_9)
- net GPIO_10: now reaches U6.43 (PA10)
- net GPIO_10: now also J5.10 (Pin_10)
- net VCAP2: now reaches C22.1, U6.47 (VCAP_2)
- net RVA+: now reaches C44.2, U9.5 (COMP)
- net RVAC+: now reaches C44.1, U9.8 (C/B)
- net LVA-: now reaches C19.2, U4.5 (COMP)
- net LVAC-: now reaches C19.1, U4.8 (C/B)
- net IREF: now reaches R12.1, U5.20 (IREF)
- net VCOM: now reaches C18.2, U5.21 (VCC1), U5.22 (VCOML)
- net LRCK: now reaches R11.2, U5.4 (LRCK)
- net I2SD: now reaches R10.2, U5.5 (DATA)
- net BCK: now reaches R9.2, U5.6 (BCK)
- net LVAC+: now reaches C27.1, U7.8 (C/B)
- net LVA+: now reaches C27.2, U7.5 (COMP)
- net CAP+: now reaches C4.2, U2.2 (CAP+)
- net CAP-: now reaches C4.1, U2.4 (CAP-)
- net LED_STATUS renamed LED_STATUS2
- net LED_STATUS2: now also D4.2 (A); no longer D3.2 (A)
- new net: D4.1 (K), R20.1
- no-connect marks 47 -> 36
Other:
- moved on the sheet: D3, R17, R18, R7
